Commit message: Work on SLAM

File: description/lidar.xacro (robot description, xacro)
@@ -43,5 +43,8 @@
             <plugin name="laser_controller" filename="libgazebo_ros_ray_sensor.so">
                 <ros>
-                    <argument>~/out:=scan</argument>
+                    <!--<argument>~/out:=scan</argument>-->
+                <ros>
+                    <remapping>~/out:=/scan</remapping>
+                </ros>
                 </ros>
                 <output_type>sensor_msgs/LaserScan</output_type>

File: description/robot_core.xacro (robot description, xacro)
@@ -16,4 +16,12 @@
     <!--- BASE LINK -->
     <link name="base_link">
+    </link>
+     <!-- BASE_FOOTPRINT LINK -->
+    <joint name="base_footprint_joint" type="fixed">
+        <parent link="base_link"/>
+        <child link="base_footprint"/>
+        <origin xyz="0 0 0" rpy="0 0 0"/>
+    </joint>
+    <link name="base_footprint">
     </link>
     <!-- CHASSIS LINK -->
